File: capacitive-scale/scale.sch (KiCad schematic (older format))
At the start: 6 parts, among them J101 TEST_1P, J102 TEST_1P, J103 TEST_1P, J104 TEST_1P, U101 outline, U102 scales

Commit message: Relayout capacitive scale and regenerate all Gerber files
Parts:
- U102: footprint capacitive:Capacitive_Scales200.00 -> capacitive:Capacitive_Scales320.00
Changed lines of the file:
@@
 F 0 "U102" H 5550 4250 60  0000 C CNN
 F 1 "scales" H 5550 4250 60  0000 C CNN
-F 2 "capacitive:Capacitive_Scales200.00" H 5550 4250 60  0001 C CNN
+F 2 "capacitive:Capacitive_Scales320.00" H 5550 4250 60  0001 C CNN
 F 3 "" H 5550 4250 60  0001 C CNN
 	1    5550 4250
