File: capacitive/capacitive.kicad_pcb (KiCad board)
At the start: 2 copper layers, 78 x 72 mm, 84 parts, among them J101 UL, J102 UART, J103 SWD, J104 TX_PADS, J105 RX_PAD, J106 POWER, J107 UR, J108 LL, J109 LR, Q101 RU1C002ZPTCL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

Commit message: Relayout capacitive scale and regenerate all Gerber files
Parts:
- moved J107 40.0 mm to (100.0, 80.0)
- moved J109 40.0 mm to (100.0, 120.0)
Changed lines of the file:
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@@
   )
   (setup
-    (last_trace_width 0.6)
+    (last_trace_width 0.1524)
     (user_trace_width 0.2)
     (user_trace_width 0.3)
@@
       (net 34 "Net-(C124-Pad2)") (solder_mask_margin 0.05))
   )
-  (module capacitive:Slide_Drill_Left (layer F.Cu)
-    (at 100 80)
-    (fp_text reference J101 (at 11.05 -0.05 90) (layer F.SilkS) hide
-      (effects (font (size 1 1) (thickness 0.15)))
-    )
-    (fp_text value UL (at 0 -0.5) (layer F.Fab)
-      (effects (font (size 1 1) (thickness 0.15)))
-    )
-    (pad 1 thru_hole circle (at -20.5149 0) (size 4.175 4.175) (drill 3.175) (layers *.Cu *.Mask)
-      (net 2 GND))
-  )
   (module Socket_Strips:Socket_Strip_Straight_2x03_Pitch2.54mm_SMD (layer F.Cu)
     (at 104.1 65.4 45)
@@
     )
   )
-  (module capacitive:Slide_Drill_Right (layer F.Cu)
-    (at 100 120)
-    (fp_text reference J107 (at 11.05 -0.05 90) (layer F.SilkS) hide
-      (effects (font (size 1 1) (thickness 0.15)))
-    )
-    (fp_text value UR (at 0 -0.5) (layer F.Fab)
-      (effects (font (size 1 1) (thickness 0.15)))
-    )
-    (pad 1 thru_hole circle (at 14.9025 0) (size 4.175 4.175) (drill 3.175) (layers *.Cu *.Mask)
-      (net 2 GND))
-  )
-  (module capacitive:Slide_Drill_Left (layer F.Cu)
-    (at 100 120)
-    (fp_text reference J108 (at 11.05 -0.05 90) (layer F.SilkS) hide
-      (effects (font (size 1 1) (thickness 0.15)))
-    )
-    (fp_text value LL (at 0 -0.5) (layer F.Fab)
-      (effects (font (size 1 1) (thickness 0.15)))
-    )
-    (pad 1 thru_hole circle (at -20.5149 0) (size 4.175 4.175) (drill 3.175) (layers *.Cu *.Mask)
-      (net 2 GND))
-  )
-  (module capacitive:Slide_Drill_Right (layer F.Cu)
-    (at 100 80)
-    (fp_text reference J109 (at 11.05 -0.05 90) (layer F.SilkS) hide
-      (effects (font (size 1 1) (thickness 0.15)))
-    )
-    (fp_text value LR (at 0 -0.5) (layer F.Fab)
-      (effects (font (size 1 1) (thickness 0.15)))
-    )
-    (pad 1 thru_hole circle (at 14.9025 0) (size 4.175 4.175) (drill 3.175) (layers *.Cu *.Mask)
-      (net 2 GND))
-  )
   (module Capacitors_SMD:C_1210_HandSoldering (layer F.Cu)
     (at 133.81 82.52 90)
@@
     )
   )
+  (module capacitive:Slide_Drill_Left (layer F.Cu)
+    (at 100 80)
+    (fp_text reference J101 (at 11.05 -0.05 90) (layer F.SilkS) hide
+      (effects (font (size 1 1) (thickness 0.15)))
+    )
+    (fp_text value UL (at 0 -0.5) (layer F.Fab)
+      (effects (font (size 1 1) (thickness 0.15)))
+    )
+    (pad 1 thru_hole circle (at -20.5149 0) (size 4.175 4.175) (drill 3.175) (layers *.Cu *.Mask)
+      (net 2 GND))
+  )
+  (module capacitive:Slide_Drill_Right (layer F.Cu)
+    (at 100 80)
+    (fp_text reference J107 (at 11.05 -0.05 90) (layer F.SilkS) hide
+      (effects (font (size 1 1) (thickness 0.15)))
+    )
+    (fp_text value UR (at 0 -0.5) (layer F.Fab)
+      (effects (font (size 1 1) (thickness 0.15)))
+    )
+    (pad 1 thru_hole circle (at 14.9025 0) (size 4.175 4.175) (drill 3.175) (layers *.Cu *.Mask)
+      (net 2 GND))
+  )
+  (module capacitive:Slide_Drill_Left (layer F.Cu)
+    (at 100 120)
+    (fp_text reference J108 (at 11.05 -0.05 90) (layer F.SilkS) hide
+      (effects (font (size 1 1) (thickness 0.15)))
+    )
+    (fp_text value LL (at 0 -0.5) (layer F.Fab)
+      (effects (font (size 1 1) (thickness 0.15)))
+    )
+    (pad 1 thru_hole circle (at -20.5149 0) (size 4.175 4.175) (drill 3.175) (layers *.Cu *.Mask)
+      (net 2 GND))
+  )
+  (module capacitive:Slide_Drill_Right (layer F.Cu)
+    (at 100 120)
+    (fp_text reference J109 (at 11.05 -0.05 90) (layer F.SilkS) hide
+      (effects (font (size 1 1) (thickness 0.15)))
+    )
+    (fp_text value LR (at 0 -0.5) (layer F.Fab)
+      (effects (font (size 1 1) (thickness 0.15)))
+    )
+    (pad 1 thru_hole circle (at 14.9025 0) (size 4.175 4.175) (drill 3.175) (layers *.Cu *.Mask)
+      (net 2 GND))
+  )
   (gr_arc (start 141 120) (end 149 120) (angle 90) (layer Edge.Cuts) (width 0.15))

Commit message: Fix reverse voltage MOSFET probably
Parts:
- moved D102 0.22 mm to (145.1, 62.5), turned to 90 degrees
- turned Q101 to 180 degrees
Connections:
- Q101 pad 2: +5V -> Net-(C115-Pad1)
- Q101 pad 3: Net-(C115-Pad1) -> +5V
Routing:
- net GND: track 426.2 -> 430.9 mm, vias 23 -> 24
- net +5V: track 48.1 -> 51.5 mm
- net Net-(C115-Pad1): track 11.4 -> 12.2 mm
Changed lines of the file:
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@@
     (thickness 1.6)
     (drawings 9)
-    (tracks 800)
+    (tracks 807)
     (zones 0)
     (modules 84)
@@
   )
   (setup
-    (last_trace_width 0.1524)
+    (last_trace_width 0.45)
     (user_trace_width 0.2)
     (user_trace_width 0.3)
@@
   )
   (module capacitive:SOD-923 (layer F.Cu)
-    (at 144.92 62.63 270)
-    (fp_text reference D102 (at 0.02 -1.18 270) (layer F.SilkS)
+    (at 145.1 62.5 90)
+    (fp_text reference D102 (at 0.02 -1.18 90) (layer F.SilkS)
       (effects (font (size 1 1) (thickness 0.15)))
     )
-    (fp_text value ESD9X5.0ST5G (at 0 -1.1 270) (layer F.Fab)
+    (fp_text value ESD9X5.0ST5G (at 0 -1.1 90) (layer F.Fab)
       (effects (font (size 1 1) (thickness 0.15)))
     )
@@
     (fp_line (start 0 0) (end -0.15 0) (layer F.SilkS) (width 0.15))
     (fp_line (start 0 -0.1) (end 0 0.1) (layer F.SilkS) (width 0.15))
-    (pad 1 smd rect (at -0.42 0 270) (size 0.36 0.25) (layers F.Cu F.Paste F.Mask)
+    (pad 1 smd rect (at -0.42 0 90) (size 0.36 0.25) (layers F.Cu F.Paste F.Mask)
       (net 9 +5V))
-    (pad 2 smd rect (at 0.42 0 270) (size 0.36 0.25) (layers F.Cu F.Paste F.Mask)
+    (pad 2 smd rect (at 0.42 0 90) (size 0.36 0.25) (layers F.Cu F.Paste F.Mask)
       (net 2 GND))
   )
   (module capacitive:Rohm_UMT3F (layer F.Cu)
-    (at 142.87 62.55 90)
-    (fp_text reference Q101 (at 2.1396 -0.02802 180) (layer F.SilkS)
+    (at 142.87 62.55 180)
+    (fp_text reference Q101 (at 2.1396 -0.02802 270) (layer F.SilkS)
       (effects (font (size 1 1) (thickness 0.15)))
     )
-    (fp_text value RU1C002ZPTCL (at 0 -2.75 90) (layer F.Fab)
+    (fp_text value RU1C002ZPTCL (at 0 -2.75 180) (layer F.Fab)
       (effects (font (size 1 1) (thickness 0.15)))
     )
@@
     (fp_line (start -1.3 -0.9) (end -1.3 -0.4) (layer F.SilkS) (width 0.15))
     (fp_line (start -1.3 -0.9) (end -0.8 -0.9) (layer F.SilkS) (width 0.15))
-    (pad 3 smd rect (at 0 -0.8 90) (size 0.8 0.9) (layers F.Cu F.Paste F.Mask)
-      (net 8 "Net-(C115-Pad1)"))
-    (pad 2 smd rect (at 0.65 0.8 90) (size 0.8 0.9) (layers F.Cu F.Paste F.Mask)
+    (pad 3 smd rect (at 0 -0.8 180) (size 0.8 0.9) (layers F.Cu F.Paste F.Mask)
       (net 9 +5V))
-    (pad 1 smd rect (at -0.65 0.8 90) (size 0.8 0.9) (layers F.Cu F.Paste F.Mask)
+    (pad 2 smd rect (at 0.65 0.8 180) (size 0.8 0.9) (layers F.Cu F.Paste F.Mask)
+      (net 8 "Net-(C115-Pad1)"))
+    (pad 1 smd rect (at -0.65 0.8 180) (size 0.8 0.9) (layers F.Cu F.Paste F.Mask)
       (net 2 GND))
   )
@@
   (segment (start 119.26 67.98) (end 117.41 67.98) (width 0.6) (layer F.Cu) (net 1))
   (segment (start 106.007178 60.707827) (end 104.892965 61.82204) (width 0.6) (layer F.Cu) (net 1))
+  (segment (start 145.1 62.08) (end 143.85 62.08) (width 0.45) (layer F.Cu) (net 2))
+  (segment (start 143.85 62.08) (end 143.52 61.75) (width 0.45) (layer F.Cu) (net 2))
+  (segment (start 143.1 60.5) (end 140.28 63.32) (width 0.6) (layer B.Cu) (net 2))
+  (segment (start 140.28 63.32) (end 140.28 67.28) (width 0.6) (layer B.Cu) (net 2))
+  (segment (start 143.52 61.75) (end 143.52 60.92) (width 0.6) (layer F.Cu) (net 2))
+  (segment (start 143.52 60.92) (end 143.1 60.5) (width 0.6) (layer F.Cu) (net 2))
+  (via (at 143.1 60.5) (size 0.6858) (drill 0.3302) (layers F.Cu B.Cu) (net 2))
+  (segment (start 137.02 62.47) (end 139.13 64.58) (width 0.6) (layer F.Cu) (net 2))
   (segment (start 130.075 65.125) (end 130.325 65.125) (width 0.6) (layer B.Cu) (net 2))
   (segment (start 130.325 65.125) (end 133.1 62.35) (width 0.6) (layer B.Cu) (net 2))
@@
   (segment (start 131.745 62.47) (end 130.4 61.125) (width 0.6) (layer F.Cu) (net 2))
   (segment (start 130.4 61.125) (end 130.4 61) (width 0.6) (layer F.Cu) (net 2))
-  (segment (start 139.13 64.58) (end 142.29 64.58) (width 0.6) (layer F.Cu) (net 2))
-  (segment (start 142.29 64.58) (end 143.67 63.2) (width 0.6) (layer F.Cu) (net 2))
   (segment (start 135.95 62.47) (end 137.02 62.47) (width 0.6) (layer F.Cu) (net 2))
-  (segment (start 137.02 62.47) (end 139.13 64.58) (width 0.6) (layer F.Cu) (net 2))
-  (segment (start 144.92 63.05) (end 143.82 63.05) (width 0.45) (layer F.Cu) (net 2))
-  (segment (start 143.82 63.05) (end 143.67 63.2) (width 0.45) (layer F.Cu) (net 2))
   (via (at 115 110.95) (size 0.6858) (drill 0.3302) (layers F.Cu B.Cu) (net 2))
   (segment (start 117.8 107.5) (end 117.8 104.79) (width 0.45) (layer F.Cu) (net 2))
@@
   (segment (start 88.857193 76.3649) (end 83.7 81.522093) (width 0.3) (layer F.Cu) (net 7))
   (segment (start 83.7 81.522093) (end 83.7 87) (width 0.3) (layer F.Cu) (net 7))
+  (segment (start 142.22 61.75) (end 140.3 61.75) (width 0.6) (layer F.Cu) (net 8))
+  (segment (start 140.3 61.75) (end 139.13 60.58) (width 0.6) (layer F.Cu) (net 8))
   (segment (start 135.95 61.52) (end 134.980678 61.52) (width 0.6) (layer F.Cu) (net 8))
   (segment (start 134.980678 61.52) (end 134.717599 61.783079) (width 0.6) (layer F.Cu) (net 8))
@@
   (segment (start 136.89 60.58) (end 135.95 61.52) (width 0.6) (layer F.Cu) (net 8))
   (segment (start 139.13 60.58) (end 140.1 60.58) (width 0.6) (layer F.Cu) (net 8))
-  (segment (start 140.1 60.58) (end 142.07 62.55) (width 0.6) (layer F.Cu) (net 8))
-  (segment (start 145.86 62.870678) (end 145.86 63.94) (width 0.6) (layer F.Cu) (net 9))
-  (segment (start 145.86 63.94) (end 144.51 65.29) (width 0.6) (layer F.Cu) (net 9))
+  (segment (start 145.8 61.795678) (end 145.8 62.85) (width 0.45) (layer F.Cu) (net 9))
+  (segment (start 145.8 62.85) (end 145.1 63.55) (width 0.45) (layer F.Cu) (net 9))
+  (segment (start 140.847599 59.127599) (end 143.131921 59.127599) (width 0.45) (layer F.Cu) (net 9))
+  (segment (start 143.131921 59.127599) (end 145.8 61.795678) (width 0.45) (layer F.Cu) (net 9))
+  (segment (start 145.1 62.92) (end 145.1 63.55) (width 0.45) (layer F.Cu) (net 9))
+  (segment (start 145.1 63.55) (end 144.95 63.7) (width 0.45) (layer F.Cu) (net 9))
+  (segment (start 143.87 63.35) (end 144.22 63.7) (width 0.6) (layer F.Cu) (net 9))
+  (segment (start 144.22 63.7) (end 144.51 63.99) (width 0.6) (layer F.Cu) (net 9))
+  (segment (start 144.95 63.7) (end 144.22 63.7) (width 0.45) (layer F.Cu) (net 9))
+  (segment (start 142.87 63.35) (end 143.87 63.35) (width 0.6) (layer F.Cu) (net 9))
+  (segment (start 144.51 63.99) (end 144.51 65.29) (width 0.6) (layer F.Cu) (net 9))
   (segment (start 144.51 65.29) (end 144.51 66.89) (width 0.6) (layer F.Cu) (net 9))
-  (segment (start 144.92 62.21) (end 145.199322 62.21) (width 0.6) (layer F.Cu) (net 9))
-  (segment (start 145.199322 62.21) (end 145.86 62.870678) (width 0.6) (layer F.Cu) (net 9))
   (segment (start 125.95 60.31) (end 127.4 60.31) (width 0.6) (layer F.Cu) (net 9))
-  (segment (start 140.847599 59.127599) (end 143.62 61.9) (width 0.6) (layer F.Cu) (net 9))
   (segment (start 127.4 60.31) (end 128.582401 59.127599) (width 0.6) (layer F.Cu) (net 9))
   (segment (start 128.582401 59.127599) (end 140.847599 59.127599) (width 0.6) (layer F.Cu) (net 9))
-  (segment (start 143.62 61.9) (end 143.67 61.9) (width 0.6) (layer F.Cu) (net 9))
-  (segment (start 144.92 62.21) (end 143.98 62.21) (width 0.45) (layer F.Cu) (net 9))
-  (segment (start 143.98 62.21) (end 143.67 61.9) (width 0.45) (layer F.Cu) (net 9))
   (segment (start 113.88 59.007599) (end 124.647599 59.007599) (width 0.6) (layer F.Cu) (net 9))
   (segment (start 124.647599 59.007599) (end 125.95 60.31) (width 0.6) (layer F.Cu) (net 9))
